File: electrical/apollo-pressure-sensor-breakout/TE-MS5837-breakout.sch (EAGLE design)
At the start: 12 parts, among them U1 TE-MS5837, X1 RJ45-8-2-CONEC-1, X2 M04X2

Commit message: resize TE board, add mounting holes
Changed lines of the file:
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@@
 <?xml version="1.0" encoding="utf-8"?>
 <!DOCTYPE eagle SYSTEM "eagle.dtd">
-<eagle version="7.6.0">
+<eagle version="9.3.0">
 <drawing>
 <settings>
 <setting alwaysvectorfont="no"/>
+<setting keepoldvectorfont="yes"/>
 <setting verticaltext="up"/>
 </settings>
@@
 <instance part="JP3" gate="G$1" x="91.44" y="-7.62" smashed="yes"/>
 <instance part="JP4" gate="G$1" x="96.52" y="-7.62" smashed="yes"/>
-<instance part="U1" gate="G$1" x="66.04" y="53.34"/>
+<instance part="U1" gate="G$1" x="66.04" y="53.34" smashed="yes">
+<attribute name="NAME" x="55.88" y="43.18" size="1.778" layer="95"/>
+<attribute name="VALUE" x="55.88" y="40.64" size="1.778" layer="96"/>
+</instance>
 </instances>
 <busses>
