File: electrical/apollo-ctrl-v4/ctrl-pico.brd (EAGLE design)
At the start: 88.6 x 88.9 mm, 47 parts, among them J1 ESP32-PICO-KIT, J2 DNP, J3 DNP, J4 DNP, J6 DISPLAY_RIGHT, J7 DISPLAY_LEFT, Q1 SOT23-3, U1 DNP (24LC01)

Commit message: DRC error-free
Routing:
- net GND: track 50.2 -> 46.4 mm
- net GPIO23: track 134.6 -> 133.7 mm
Changed lines of the file:
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@@
 <via x="10.795" y="2.54" extent="1-16" drill="0.45"/>
 <via x="46.99" y="1.905" extent="1-16" drill="0.45"/>
-<wire x1="17.78" y1="78.87" x2="16.51" y2="77.6" width="0.2032" layer="16"/>
-<wire x1="16.51" y1="77.6" x2="16.51" y2="75.565" width="0.2032" layer="16"/>
 <wire x1="27.94" y1="78.87" x2="29.21" y2="77.6" width="0.2032" layer="1"/>
 <wire x1="29.21" y1="77.6" x2="29.21" y2="75.565" width="0.2032" layer="1"/>
-<wire x1="32.52550625" y1="77.5238" x2="31.8262" y2="76.82449375" width="0.2032" layer="1"/>
+<wire x1="32.52550625" y1="77.5238" x2="31.75" y2="76.74829375" width="0.2032" layer="1"/>
 <wire x1="35.56" y1="78.87" x2="34.2138" y2="77.5238" width="0.2032" layer="1"/>
 <wire x1="34.2138" y1="77.5238" x2="32.52550625" y2="77.5238" width="0.2032" layer="1"/>
-<wire x1="31.8262" y1="76.82449375" x2="31.8262" y2="75.6412" width="0.2032" layer="1"/>
+<wire x1="31.75" y1="76.74829375" x2="31.75" y2="75.6158" width="0.2032" layer="1"/>
 <wire x1="53.34" y1="78.87" x2="54.61" y2="77.6" width="0.2032" layer="1"/>
 <wire x1="54.61" y1="77.6" x2="54.61" y2="75.565" width="0.2032" layer="1"/>
@@
 <polygon width="0.2032" layer="1" isolate="0.3048">
 <vertex x="16.51" y="80.645"/>
-<vertex x="16.51" y="77.47"/>
 <vertex x="10.795" y="77.47"/>
 <vertex x="3.81" y="70.485"/>
@@
 <wire x1="33.655" y1="13.97" x2="42.28" y2="13.97" width="0.2032" layer="1"/>
 <wire x1="42.28" y1="13.97" x2="43.18" y2="13.07" width="0.2032" layer="1"/>
-<wire x1="26.67" y1="41.275" x2="26.67" y2="27.71798125" width="0.2032" layer="16"/>
-<wire x1="31.7483" y1="15.8767" x2="31.7483" y2="22.63968125" width="0.2032" layer="16"/>
+<wire x1="26.67" y1="41.275" x2="26.67" y2="27.46398125" width="0.2032" layer="16"/>
+<wire x1="31.7483" y1="15.8767" x2="31.7483" y2="22.38568125" width="0.2032" layer="16"/>
 <wire x1="33.655" y1="13.97" x2="31.7483" y2="15.8767" width="0.2032" layer="16"/>
-<wire x1="31.7483" y1="22.63968125" x2="26.67" y2="27.71798125" width="0.2032" layer="16"/>
+<wire x1="31.7483" y1="22.38568125" x2="26.67" y2="27.46398125" width="0.2032" layer="16"/>
 </signal>
 <signal name="VMON">
@@
 <wire x1="50.8" y1="1.27" x2="73.025" y2="1.27" width="0.2032" layer="1"/>
 <wire x1="73.025" y1="1.27" x2="78.105" y2="6.35" width="0.2032" layer="1"/>
-<wire x1="79.6036" y1="43.18" x2="78.74" y2="43.18" width="0.2032" layer="1"/>
 <wire x1="79.6036" y1="43.18" x2="78.105" y2="43.18" width="0.2032" layer="1"/>
 <wire x1="78.105" y1="43.18" x2="60.325" y2="43.18" width="0.2032" layer="1"/>
